Commit message: corrected joint axis and service name

File: catkin_ws/src/my_robot/urdf/my_robot.xacro (robot description, xacro)
@@ -161,5 +161,5 @@
       <child link="right_wheel" />
       <parent link="chassis" />
-      <axis xyz="0 -1 0" rpy="0 0 0" />
+      <axis xyz="0 1 0" rpy="0 0 0" />
       <limit effort="10000" velocity="1000" />
       <dynamics damping="1.0" friction="1.0" />

Commit message: updated robot model

File: catkin_ws/src/my_robot/urdf/my_robot.xacro (robot description, xacro)
@@ -23,5 +23,5 @@
       <origin xyz="0 0 0" rpy="0 0 0" />
       <geometry>
-        <box size=".4 .2 .1" />
+        <box size=".6 .4 .1" />
       </geometry>
     </collision>
@@ -29,9 +29,9 @@
       <origin xyz="0 0 0" rpy="0 0 0" />
       <geometry>
-        <box size=".4 .2 .1" />
+        <box size=".6 .4 .1" />
       </geometry>
     </visual>
    <collision name="back_caster_collision">
-      <origin xyz="-0.15 0 -0.05" rpy="0 0 0" />
+      <origin xyz="0.2 -0.1 -0.05" rpy="0 0 0" />
       <geometry>
         <sphere radius="0.0499" />
@@ -39,5 +39,5 @@
     </collision>
    <visual name="back_caster_visual">
-      <origin xyz="-0.15 0 -0.05" rpy="0 0 0" />
+      <origin xyz="0.2 -0.1 -0.05" rpy="0 0 0" />
       <geometry>
         <sphere radius="0.0499" />
@@ -45,5 +45,5 @@
     </visual>
    <collision name="front_caster_collision">
-      <origin xyz="0.15 0 -0.05" rpy="0 0 0" />
+      <origin xyz="0.2 0.1 -0.05" rpy="0 0 0" />
       <geometry>
         <sphere radius="0.0499" />
@@ -51,5 +51,5 @@
     </collision>
    <visual name="front_caster_visual">
-      <origin xyz="0.15 0 -0.05" rpy="0 0 0" />
+      <origin xyz="0.2 0.1 -0.05" rpy="0 0 0" />
       <geometry>
         <sphere radius="0.0499" />
@@ -103,4 +103,146 @@
     </collision>
   </link>
+<link name="lf_support">
+    <inertial>
+        <mass value="0.5" />
+        <origin xyz="0 0 0" rpy="0 0 0" />
+        <inertia
+            ixx="0.1" ixy="0" ixz="0"
+            iyy="0.1" iyz="0"
+            izz="0.1" />
+        </inertial>
+    <visual name="lf_support_visual">
+        <origin xyz="0 0 0" rpy="0 0 0"/>
+        <geometry>
+            <cylinder radius="0.015" length="0.12" />
+        </geometry>
+    </visual>
+    <collision name="lf_support_collision">
+        <origin xyz="0 0 0" rpy="0 0 0"/>
+        <geometry>
+            <cylinder radius="0.015" length="0.12" />
+        </geometry>
+    </collision>
+  </link>
+  <joint type="fixed" name="lf_d_support_joint">
+      <origin xyz="0.1 0.15 0.1" rpy="0 0 0" />
+      <child link="lf_support" />
+      <parent link="chassis" />
+      <axis xyz="0 0 0" rpy="0 0 0" />
+  </joint>
+<link name="lb_support">
+    <inertial>
+        <mass value="0.5" />
+        <origin xyz="0 0 0" rpy="0 0 0" />
+        <inertia
+            ixx="0.1" ixy="0" ixz="0"
+            iyy="0.1" iyz="0"
+            izz="0.1" />
+        </inertial>
+    <visual name="lb_support_visual">
+        <origin xyz="0 0 0" rpy="0 0 0"/>
+        <geometry>
+            <cylinder radius="0.015" length="0.12" />
+        </geometry>
+    </visual>
+    <collision name="lb_support_collision">
+        <origin xyz="0 0 0" rpy="0 0 0"/>
+        <geometry>
+            <cylinder radius="0.015" length="0.12" />
+        </geometry>
+    </collision>
+  </link>
+  <joint type="fixed" name="lb_d_support_joint">
+      <origin xyz="-0.25 0.15 0.1" rpy="0 0 0" />
+      <child link="lb_support" />
+      <parent link="chassis" />
+      <axis xyz="0 0 0" rpy="0 0 0" />
+  </joint>
+<link name="rf_support">
+    <inertial>
+        <mass value="0.5" />
+        <origin xyz="0 0 0" rpy="0 0 0" />
+        <inertia
+            ixx="0.1" ixy="0" ixz="0"
+            iyy="0.1" iyz="0"
+            izz="0.1" />
+        </inertial>
+    <visual name="rf_support_visual">
+        <origin xyz="0 0 0" rpy="0 0 0"/>
+        <geometry>
+            <cylinder radius="0.015" length="0.12" />
+        </geometry>
+    </visual>
+    <collision name="rf_support_collision">
+        <origin xyz="0 0 0" rpy="0 0 0"/>
+        <geometry>
+            <cylinder radius="0.015" length="0.12" />
+        </geometry>
+    </collision>
+  </link>
+  <joint type="fixed" name="rf_d_support_joint">
+      <origin xyz="0.1 -0.15 0.1" rpy="0 0 0" />
+      <child link="rf_support" />
+      <parent link="chassis" />
+      <axis xyz="0 0 0" rpy="0 0 0" />
+  </joint>
+<link name="rb_support">
+    <inertial>
+        <mass value="0.5" />
+        <origin xyz="0 0 0" rpy="0 0 0" />
+        <inertia
+            ixx="0.1" ixy="0" ixz="0"
+            iyy="0.1" iyz="0"
+            izz="0.1" />
+        </inertial>
+    <visual name="rb_support_visual">
+        <origin xyz="0 0 0" rpy="0 0 0"/>
+        <geometry>
+            <cylinder radius="0.015" length="0.12" />
+        </geometry>
+    </visual>
+    <collision name="rb_support_collision">
+        <origin xyz="0 0 0" rpy="0 0 0"/>
+        <geometry>
+            <cylinder radius="0.015" length="0.12" />
+        </geometry>
+    </collision>
+  </link>
+  <joint type="fixed" name="rb_d_support_joint">
+      <origin xyz="-0.25 -0.15 0.1" rpy="0 0 0" />
+      <child link="rb_support" />
+      <parent link="chassis" />
+      <axis xyz="0 0 0" rpy="0 0 0" />
+  </joint>
+<link name="upper_chassis">
+    <pose>0 0 0.1 0 0 0</pose>
+    <inertial>
+      <mass value="5.0"/>
+      <origin xyz="0.0 0 0" rpy="0 0 0" />
+      <inertia
+        ixx="0.1" ixy="0" ixz="0"
+        iyy="0.1" iyz="0"
+        izz="0.1"
+      />
+    </inertial>
+    <collision name="upper_chassis_collision">
+      <origin xyz="0 0 0" rpy="0 0 0" />
+      <geometry>
+        <box size=".4 .4 .04" />
+      </geometry>
+    </collision>
+    <visual name='upper_chassis_visual'>
+      <origin xyz="0 0 0" rpy="0 0 0" />
+      <geometry>
+        <box size=".4 .4 .04" />
+      </geometry>
+    </visual>
+  </link>
+  <joint type="fixed" name="lf_u_support">
+      <origin xyz="-0.18 -0.15 0.05" rpy="0 0 0" />
+      <child link="upper_chassis" />
+      <parent link="lf_support" />
+      <axis xyz="0 0 0" rpy="0 0 0" />
+  </joint>
   <link name="camera">
       <inertial>
@@ -150,5 +292,5 @@
   </link>
   <joint type="continuous" name="left_wheel_hinge">
-      <origin xyz="0 0.15 0" rpy="0 0 0" />
+      <origin xyz="-0.15 0.25 0" rpy="0 0 0" />
       <child link="left_wheel" />
       <parent link="chassis" />
@@ -158,5 +300,5 @@
   </joint>
   <joint type="continuous" name="right_wheel_hinge">
-      <origin xyz="0 -0.15 0" rpy="0 0 0" />
+      <origin xyz="-0.15 -0.25 0" rpy="0 0 0" />
       <child link="right_wheel" />
       <parent link="chassis" />
@@ -166,5 +308,5 @@
   </joint>
   <joint type="fixed" name="camera_joint">
-      <origin xyz="0.2 0 0" rpy="0 0 0" />
+      <origin xyz="0.3 0 0" rpy="0 0 0" />
       <child link="camera" />
       <parent link="chassis" />
@@ -172,8 +314,35 @@
   </joint>
   <joint type="fixed" name="hokuyo_joint">
-      <origin xyz="0.15 0 0.1" rpy="0 0 0" />
+      <origin xyz="0.05 0 0.2" rpy="0 0 0" />
       <child link="hokuyo" />
       <parent link="chassis" />
       <axis xyz="0 1 0" rpy="0 0 0" />
   </joint>
+  <gazebo reference="left_wheel">
+    <material>Gazebo/Black</material>
+  </gazebo>
+  <gazebo reference="right_wheel">
+    <material>Gazebo/Black</material>
+  </gazebo>
+  <gazebo reference="chassis">
+    <material>Gazebo/White</material>
+  </gazebo>
+  <gazebo reference="lf_support">
+    <material>Gazebo/Black</material>
+  </gazebo>
+  <gazebo reference="lb_support">
+    <material>Gazebo/Black</material>
+  </gazebo>
+  <gazebo reference="rb_support">
+    <material>Gazebo/Black</material>
+  </gazebo>
+  <gazebo reference="rf_support">
+    <material>Gazebo/Black</material>
+  </gazebo>
+  <gazebo reference="upper_chassis">
+    <material>Gazebo/White</material>
+  </gazebo>
+  <gazebo reference="camera">
+    <material>Gazebo/Red</material>
+  </gazebo>
 </robot>

Commit message: tuned amcl parameters. simulation running fine

File: catkin_ws/src/my_robot/urdf/my_robot.xacro (robot description, xacro)
@@ -103,34 +103,4 @@
     </collision>
   </link>
-<link name="upper_chassis">
-    <pose>0 0 0.1 0 0 0</pose>
-    <inertial>
-      <mass value="1.0"/>
-      <origin xyz="0.0 0 0" rpy="0 0 0" />
-      <inertia
-        ixx="0.1" ixy="0" ixz="0"
-        iyy="0.1" iyz="0"
-        izz="0.1"
-      />
-    </inertial>
-    <collision name="upper_chassis_collision">
-      <origin xyz="0 0 0" rpy="0 0 0" />
-      <geometry>
-        <box size=".1 .1 .04" />
-      </geometry>
-    </collision>
-    <visual name='upper_chassis_visual'>
-      <origin xyz="0 0 0" rpy="0 0 0" />
-      <geometry>
-        <box size=".1 .1 .04" />
-      </geometry>
-    </visual>
-  </link>
-  <joint type="fixed" name="lf_u_support">
-      <origin xyz="0.15 0 0.05" rpy="0 0 0" />
-      <child link="upper_chassis" />
-      <parent link="chassis" />
-      <axis xyz="0 1 0" rpy="0 0 0" />
-  </joint>
   <link name="camera">
       <inertial>
